File: pcb/STM32U545RETxQ.kicad_sch (KiCad schematic)
At the start: 20 parts, among them U3 STM32U545RETxQ

Commit message: Updated Schematics
Completed Schematics for Test Bed, updated pcb
Parts:
- renumbered C12 to C10, C13 to C11, C14 to C12, C15 to C13, C4 to C2, C5 to C3, C6 to C4, C7 to C5, C8 to C6, C9 to C7, C10 to C8, C11 to C9, TP_3V3_mcu to TP_3V3_mcu1, TP_ADC_BAT_DIV to TP_ADC_BAT_DIV1, TP_BOOT0 to TP_BOOT1, TP_NRST to TP_NRST1, TP_SD_EJECT to TP_SD_EJECT1, TP_VUSB to TP_VUSB1
