File: pcb/Battery_testbed.kicad_sch (KiCad schematic)
At the start: 12 parts, among them U5 MIC5504-3.3YM5, U6 MCP73831-2-OT

Commit message: Updated Schematics
Completed Schematics for Test Bed, updated pcb
Parts:
- added TP_3V3_reg1: TestPoint, TestPoint:TestPoint_Loop_D2.54mm_Drill1.5mm_Beaded, symbol Connector:TestPoint
- renumbered C11 to C18, C13 to C19, C10 to C20, C12 to C21, D1 to D3, D2 to D4, R3 to R16, R4 to R17, R5 to R18, U5 to U7
Connections:
- net +3.3V: now also TP_3V3_reg1.1
- net V_{BAT}: no longer C19.1, U7.1 (VIN), U7.3 (EN)
- net +5V renamed +5V_USB
- net +5V_USB: no longer U6.4 (V_{DD})
- new net V_USB: U6.4 (V_{DD})
- new net V_{mux}: C19.1, U7.1 (VIN), U7.3 (EN)

Commit message: Pre-fab update
Pre fab update
Parts:
- removed TP_3V3_reg1: TestPoint, TestPoint:TestPoint_Loop_D2.54mm_Drill1.5mm_Beaded, symbol Connector:TestPoint
- added Pwr_Mux_ST1, V_{mux}1: TestPoint, TestPoint:TestPoint_Loop_D2.54mm_Drill1.5mm_Beaded, symbol Connector:TestPoint
- added R1: 300k, Resistor_SMD:R_0603_1608Metric_Pad0.98x0.95mm_HandSolder, symbol Device:R_US
- added R2: 100k, Resistor_SMD:R_0603_1608Metric_Pad0.98x0.95mm_HandSolder, symbol Device:R_US
- added R4: 10k, Resistor_SMD:R_0603_1608Metric, symbol Device:R_US
- added U1: TPS2116DRL, Package_TO_SOT_SMD:SOT-583-8, symbol Power_Management:TPS2116DRL
Connections:
- net V_USB is gone; now on net +5V_USB: U6.4 (V_{DD})
- net +3.3V: now also R4.1
- net +5V_USB: now also R1.2, U1.3 (VIN1), U1.5 (MODE)
- net GNDD: now also R2.1, U1.1 (GND)
- net V_{BAT}: now also U1.6 (VIN2)
- net V_{mux}: now also U1.2 (VOUT), U1.7 (VOUT), V_{mux}1.1
- new net: R1.1, R2.2, U1.4 (PR1)
- new net: Pwr_Mux_ST1.1, R4.2, U1.8 (ST)
