File: pcb/control-module.kicad_sch (KiCad schematic)
At the start: 29 parts, among them J1 Screw_Terminal_01x06, J2 Conn_01x07_Pin, SW1 SW_DIP_x04, U1 TPS2116DRL

Commit message: Pre-fab update
Pre fab update
Parts:
- removed J2: Conn_01x07_Pin, Connector_PinHeader_2.54mm:PinHeader_1x07_P2.54mm_Vertical, symbol Connector:Conn_01x07_Pin
- removed R1: 300k, Resistor_SMD:R_0603_1608Metric_Pad0.98x0.95mm_HandSolder, symbol Device:R_US
- removed R2: 100k, Resistor_SMD:R_0603_1608Metric_Pad0.98x0.95mm_HandSolder, symbol Device:R_US
- removed R4: 10k, Resistor_SMD:R_0603_1608Metric, symbol Device:R_US
- removed TP_Power_Mux_STAT1, TP_V_{BAT}1, TP_V_{mux}1: TestPoint, TestPoint:TestPoint_Loop_D2.54mm_Drill1.5mm_Beaded, symbol Connector:TestPoint
- removed U1: TPS2116DRL, Package_TO_SOT_SMD:SOT-583-8, symbol Power_Management:TPS2116DRL
- added JP3, JP4: SolderJumper_2_Open, Jumper:SolderJumper-2_P1.3mm_Open_RoundedPad1.0x1.5mm, symbol Jumper:SolderJumper_2_Open
- renumbered TP_BATT1 to BATT1, TP_BAT_SENSE_MID1 to BAT_SENSE_MID1
Connections:
- net +BATT is gone; now on net V_{BAT}: BATT1.1, RN1.1 (R1.1)
- net USB-C/V_USB renamed USB-C/+5V_USB
- new net Ublox_GPS_module/GPS_RX: JP4.2 (B)
- new net Ublox_GPS_module/GPS_TX: JP3.1 (A)
- new net radio_RX: JP4.1 (A)
- new net radio_TX: JP3.2 (B)
Other:
- sheet Battery ports: added none; removed V_{mux}
- sheet MCU ports: added SPI3_CS, SPI3_MISO, SPI3_MOSI, SPI3_SCK; removed none
- sheet STLink ports: added NRST_radio, STLink_radio_RX, STLink_radio_TX, SWCLK_radio, SWDIO_radio, SWO_radio; removed none
- sheet USB-C ports: added +5V_USB; removed V_USB
- sheet Ublox_GPS_module ports: added GPS_RX, GPS_TX, TIMEPULSE_OUT; removed none
- sheet transmitter ports: added NRST_radio, SPI1_CS_radio, SPI1_MISO_radio, SPI1_MOSI_radio, SPI1_SCK_radio, SWCLK_radio, SWDIO_radio, SWO_radio, TIMEPULSE_IN, USART1_RX_radio, USART1_TX_radio; removed none
